File: pcb/lamp_rev_b_controller/lamp_rev_b_controller.kicad_pcb (KiCad board)
At the start: 4 copper layers, 118 x 94 mm, 155 parts, among them J1 TYPE-C 3.1 MT 16P, J10 2-pin NTC header, J11 2-pin NTC header, J12 DB128H-5.08-2P-BK-S, J13 DB128H-5.08-2P-BK-S, J15 DB128H-5.08-2P-BK-S, J16 LED NTC/ID header, J17 External camera sync header, J18 SPI/FIFO camera module header, J19 Lid/cartridge/cutoff interloc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, J2 DB128H-5.08-2P-BK-S, J20 Fan PWM/tach header, J21 2x3 UART/programming header, J22 I2C expansion header, J23 Analog optical diagnostic hea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, J24 DB128H-5.08-2P high-current h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, J4 2-pin NTC header, J5 2-pin NTC header, J6 2-pin NTC header, J7 2-pin NTC header, J8 2-pin NTC header, J9 2-pin NTC header, Q1 IRLB3813PBF TO-220 12V protot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, Q2 IRLB3813PBF TO-220 12V protot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, U1 ESP32-S3-WROOM-1-N16, U10 INA180A1IDBVR gain 20 LED cur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, U2 USBLC6-2SC6, U3 Diodes AP63203WU-7 fixed 3.3V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, U4 ADS1115IDGSR, U5 CD74HC4051M, U6 TC4427ACOA/TC4427EPA, U7 CUI/Bel P7805-2000-S 5V 2A 8-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, U8 Mean Well LDD-700H 700mA CC b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, U9 SN74LVC1G08DBVR LED_EXC_PWM A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

Commit message: Close Rev B HEATER_ARM local route open
Routing:
- net HEATER_ARM: track 2.59 -> 9.43 mm, vias 0 -> 2
Changed lines of the file:
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@@
     (net 70)
   )
+  (via
+    (at 86.300 56)
+    (size 0.700)
+    (drill 0.300)
+    (layers "F.Cu" "B.Cu")
+    (net 32)
+  )
+  (via
+    (at 91.300 53)
+    (size 0.700)
+    (drill 0.300)
+    (layers "F.Cu" "B.Cu")
+    (net 32)
+  )
   (segment
     (start 32.170 60.740)
@@
     (net 70)
   )
+  (segment
+    (start 87 56)
+    (end 86.300 56)
+    (width 0.250)
+    (layer "F.Cu")
+    (net 32)
+  )
+  (segment
+    (start 86.300 56)
+    (end 91.300 53)
+    (width 0.250)
+    (layer "In2.Cu")
+    (net 32)
+  )
+  (segment
+    (start 91.300 53)
+    (end 91 53)
+    (width 0.250)
+    (layer "F.Cu")
+    (net 32)
+  )
   (zone

Commit message: Close VIN_PROTECTED Rev B route
Routing:
- net VIN_PROTECTED: track 87.0 -> 109.0 mm, vias 2 -> 4
Changed lines of the file:
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@@
   )
   (via
+    (at 76 34)
+    (size 1.200)
+    (drill 0.500)
+    (layers "F.Cu" "B.Cu")
+    (net 5)
+  )
+  (via
+    (at 86 46)
+    (size 1.200)
+    (drill 0.500)
+    (layers "F.Cu" "B.Cu")
+    (net 5)
+  )
+  (via
     (at 16.500 9.500)
     (size 0.700)
@@
     (net 5)
   )
+  (segment
+    (start 76 34)
+    (end 86 34)
+    (width 1.500)
+    (layer "In2.Cu")
+    (net 5)
+  )
+  (segment
+    (start 86 34)
+    (end 86 46)
+    (width 1.500)
+    (layer "In2.Cu")
+    (net 5)
+  )
